File: tsuka60-pro.kicad_pcb (KiCad board)
At the start: 2 copper layers, 285 x 94.6 mm, 170 parts, among them J1 USB_C_Receptacle_USB2.0, J2 Conn_01x04_MountingPin, SW1 SW_Reset, U1 ATmega32U4-M, U2 SRV05-4, Y1 16MHz

Commit message: Finish traces, draft 1
Parts:
- moved D68 24.8 mm to (208.0, 167.5)
- moved D59 20.6 mm to (322.3, 148.4)
- moved R2 8.19 mm to (87.0, 123.8), turned to 180 degrees
- moved C1 3.23 mm to (108.0, 114.3)
- moved C2 3.23 mm to (102.2, 114.3)
- moved Y1 3.23 mm to (105.1, 114.3)
- moved D63 2.38 mm to (119.1, 165.1)
- moved G*** 2.33 mm to (227.7, 117.2)
- moved G*** 2.12 mm to (185.5, 117.8)
- moved G*** 1.50 mm to (206.4, 116.2)
- moved C5 1.00 mm to (87.0, 122.2), turned to 180 degrees
Connections:
- U1 pad 1: COL0 -> unconnected-(U1-Pad1)
- U1 pad 11: COL1 -> unconnected-(U1-Pad11)
- U1 pad 12: ROW2 -> ROW0
- U1 pad 21: COL3 -> ROW2
- U1 pad 22: COL2 -> COL3
- U1 pad 36: unconnected-(U1-Pad36) -> COL2
- U1 pad 37: unconnected-(U1-Pad37) -> ROW3
- U1 pad 39: unconnected-(U1-Pad39) -> COL1
- U1 pad 40: unconnected-(U1-Pad40) -> COL0
- U1 pad 41: unconnected-(U1-Pad41) -> ROW1
- U1 pad 8: ROW0 -> unconnected-(U1-Pad8)
- U1 pad 9: ROW1 -> unconnected-(U1-Pad9)
Routing:
- net ROW4: track 250.8 -> 313.9 mm
- net 32_2: track 0.00 -> 61.7 mm, vias 0 -> 1
- net ROW3: track 219.1 -> 276.9 mm
- net ROW1: track 212.7 -> 262.0 mm, vias 0 -> 2
- net ROW2: track 205.6 -> 249.3 mm
- net COL1: track 80.3 -> 116.4 mm
- net +5V: track 74.1 -> 105.5 mm, vias 0 -> 5
- net COL0: track 74.4 -> 100.7 mm
- net COL2: track 95.1 -> 120.0 mm
- net Net-(D68-Pad2): track 6.58 -> 30.6 mm, vias 0 -> 1
- net GND: track 73.4 -> 95.8 mm
- net Net-(D30-Pad2): track 0.00 -> 13.3 mm
- net Net-(D59-Pad2): track 6.58 -> 18.1 mm
- net ROW0: track 272.9 -> 280.4 mm
- net Net-(D16-Pad2): track 0.00 -> 6.58 mm
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Other:
- board text added: "Tsuka60 Pro Rev 1 by RominRonin"
- board text removed: "Katana60 Pro Rev 1 by RominRonin"

Commit message: Update traces
Parts:
- moved D63 2.38 mm to (119.1, 167.5)
- moved D16 1.77 mm to (80.2, 111.9)
- moved SW1 0.79 mm to (100.0, 131.8)
- moved R1 0.72 mm to (96.5, 125.7)
- moved C4 0.23 mm to (97.4, 121.4)
- moved R6 0.20 mm to (83.3, 101.4)
- moved R5 0.20 mm to (81.8, 101.4)
Routing:
- net COL2: track 120.0 -> 131.7 mm, vias 0 -> 1
- net 32_2: track 61.7 -> 51.0 mm, vias 1 -> 2
- net COL0: track 100.7 -> 96.3 mm, vias 0 -> 2
- net Net-(R6-Pad2): track 15.0 -> 17.9 mm
- net Net-(D63-Pad2): track 4.20 -> 6.51 mm
- net Net-(R5-Pad2): track 15.3 -> 17.4 mm
- net ROW4: track 313.9 -> 312.1 mm
- net VCC: track 23.8 -> 22.5 mm
- net Net-(D16-Pad2): track 6.58 -> 7.84 mm
- net +5V: track 105.5 -> 104.9 mm
- net ROW1: track 262.0 -> 262.5 mm
- net Net-(D1-Pad2): vias 2 -> 1

Commit message: Update traces
Parts:
- moved D2 21.8 mm to (119.1, 91.3)
- moved D1 10.7 mm to (103.2, 91.3)
- moved D17 3.17 mm to (119.1, 110.3)
- moved D18 3.17 mm to (122.2, 110.3)
- moved D3 3.17 mm to (122.2, 91.3)
Routing:
- net ROW0: track 280.4 -> 258.8 mm
- net Net-(D2-Pad2): track 15.6 -> 32.3 mm
- net GND: track 95.6 -> 105.8 mm, vias 0 -> 2
- net Net-(D1-Pad2): track 30.1 -> 37.1 mm
- net Net-(D18-Pad2): track 6.58 -> 8.82 mm
- net Net-(D17-Pad2): track 27.1 -> 25.3 mm
- net Net-(D3-Pad2): track 6.58 -> 7.89 mm

Commit message: Made important changes to the keyboard, re-exported production files
Parts:
- added MX70_2: MX-NoLED, marbastlib-mx:SW_MX_HS_1u, B.Cu at (206.4, 165.1)
- moved S1 28.6 mm to (206.4, 165.1)
- moved D67 17.5 mm to (187.3, 167.5)
- moved D68 15.9 mm to (223.8, 167.5)
- moved D69 3.97 mm to (227.8, 167.5)
Connections:
- net Net-(D70-Pad2) renamed 70_2
- MX70 pad 1: unconnected-(MX70-Pad1) -> COL9
Routing:
- net COL9: track 240.6 -> 294.7 mm
- net 70_2: track 6.58 -> 47.7 mm
- net Net-(D67-Pad2): track 6.58 -> 16.8 mm
- net Net-(D69-Pad2): track 6.58 -> 14.6 mm, vias 0 -> 1
- net Net-(D68-Pad2): track 30.6 -> 27.5 mm
- net ROW4: track 312.1 -> 313.7 mm
